Commit message: adding the ability to use the EffortJointInterface for the ur10

File: ur_description/urdf/ur.transmission.xacro (robot description, xacro)
@@ -1,9 +1,9 @@
 <?xml version="1.0"?>
 <robot xmlns:xacro="http://www.ros.org/wiki/xacro">
-  <xacro:macro name="ur_arm_transmission" params="prefix">
+  <xacro:macro name="ur_arm_transmission" params="prefix joint_interface:=PositionJointInterface">
     <transmission name="${prefix}shoulder_pan_trans">
       <type>transmission_interface/SimpleTransmission</type>
       <joint name="${prefix}shoulder_pan_joint">
-        <hardwareInterface>PositionJointInterface</hardwareInterface>
+        <hardwareInterface>${joint_interface}</hardwareInterface>
       </joint>
       <actuator name="${prefix}shoulder_pan_motor">
@@ -14,5 +14,5 @@
       <type>transmission_interface/SimpleTransmission</type>
       <joint name="${prefix}shoulder_lift_joint">
-        <hardwareInterface>PositionJointInterface</hardwareInterface>
+        <hardwareInterface>${joint_interface}</hardwareInterface>
       </joint>
       <actuator name="${prefix}shoulder_lift_motor">
@@ -23,5 +23,5 @@
       <type>transmission_interface/SimpleTransmission</type>
       <joint name="${prefix}elbow_joint">
-        <hardwareInterface>PositionJointInterface</hardwareInterface>
+        <hardwareInterface>${joint_interface}</hardwareInterface>
       </joint>
       <actuator name="${prefix}elbow_motor">
@@ -32,5 +32,5 @@
       <type>transmission_interface/SimpleTransmission</type>
       <joint name="${prefix}wrist_1_joint">
-        <hardwareInterface>PositionJointInterface</hardwareInterface>
+        <hardwareInterface>${joint_interface}</hardwareInterface>
       </joint>
       <actuator name="${prefix}wrist_1_motor">
@@ -41,5 +41,5 @@
       <type>transmission_interface/SimpleTransmission</type>
       <joint name="${prefix}wrist_2_joint">
-        <hardwareInterface>PositionJointInterface</hardwareInterface>
+        <hardwareInterface>${joint_interface}</hardwareInterface>
       </joint>
       <actuator name="${prefix}wrist_2_motor">
@@ -50,5 +50,5 @@
       <type>transmission_interface/SimpleTransmission</type>
       <joint name="${prefix}wrist_3_joint">
-        <hardwareInterface>PositionJointInterface</hardwareInterface>
+        <hardwareInterface>${joint_interface}</hardwareInterface>
       </joint>
       <actuator name="${prefix}wrist_3_motor">

File: ur_description/urdf/ur10.urdf.xacro (robot description, xacro)
@@ -5,4 +5,5 @@
   Contributers: Jimmy Da Silva, Ajit Krisshna N L, Muhammad Asif Rana
 -->
+  <xacro:arg name="use_effort_interface" defalut="false" />
   <xacro:include filename="$(find ur_description)/urdf/ur.transmission.xacro" />
   <xacro:include filename="$(find ur_description)/urdf/ur.gazebo.xacro" />
@@ -271,5 +272,10 @@
       </collision>
     </link>
-    <xacro:ur_arm_transmission prefix="${prefix}" />
+    <xacro:if value="$(arg use_effort_interface)">
+      <xacro:ur_arm_transmission prefix="${prefix}" joint_interface="EffortJointInterface" />
+    </xacro:if>
+    <xacro:unless value="$(arg use_effort_interface)">
+      <xacro:ur_arm_transmission prefix="${prefix}" joint_interface="PositionJointInterface" />
+    </xacro:unless>
     <xacro:ur_arm_gazebo prefix="${prefix}" />
     <!-- ROS base_link to UR 'Base' Coordinates transform -->

Commit message: make joint interface configurable with xacro arg

File: ur_description/urdf/ur.transmission.xacro (robot description, xacro)
@@ -1,5 +1,26 @@
 <?xml version="1.0"?>
 <robot xmlns:xacro="http://www.ros.org/wiki/xacro">
-  <xacro:macro name="ur_arm_transmission" params="prefix joint_interface:=PositionJointInterface">
+  <xacro:arg name="use_velocity_interface" default="false" />
+  <xacro:arg name="use_effort_interface" default="false" />
+  <xacro:macro name="ur_arm_transmission" params="prefix">
+    <!-- if use_position_interface create PositionJointInterface based transmissions -->
+    <xacro:unless value="$(arg use_velocity_interface)">
+    <xacro:unless value="$(arg use_effort_interface)">
+      <!-- option1 -->
+      <xacro:ur_arm_transmission_impl prefix="${prefix}" joint_interface="PositionJointInterface" />
+    </xacro:unless>
+    </xacro:unless>
+    <!-- if use_velocity_interface create VelocityJointInterface based transmissions -->
+    <xacro:if value="$(arg use_velocity_interface)">
+      <!-- option2 -->
+      <xacro:ur_arm_transmission_impl prefix="${prefix}" joint_interface="VelocityJointInterface" />
+    </xacro:if>
+    <!-- if use_effort_interface create EffortJointInterface based transmissions -->
+    <xacro:if value="$(arg use_effort_interface)">
+      <!-- option3 -->
+      <xacro:ur_arm_transmission_impl prefix="${prefix}" joint_interface="EffortJointInterface" />
+    </xacro:if>
+  </xacro:macro>
+  <xacro:macro name="ur_arm_transmission_impl" params="prefix joint_interface">
     <transmission name="${prefix}shoulder_pan_trans">
       <type>transmission_interface/SimpleTransmission</type>

File: ur_description/urdf/ur10.urdf.xacro (robot description, xacro)
@@ -5,5 +5,5 @@
   Contributers: Jimmy Da Silva, Ajit Krisshna N L, Muhammad Asif Rana
 -->
-  <xacro:arg name="use_effort_interface" defalut="false" />
+  <xacro:arg name="joint_limited" default="false" />
   <xacro:include filename="$(find ur_description)/urdf/ur.transmission.xacro" />
   <xacro:include filename="$(find ur_description)/urdf/ur.gazebo.xacro" />
@@ -54,5 +54,5 @@
     </inertial>
   </xacro:macro>
-  <xacro:macro name="ur10_robot" params="prefix joint_limited">
+  <xacro:macro name="ur10_robot" params="prefix">
     <link name="${prefix}base_link" >
       <visual>
@@ -78,8 +78,8 @@
       <origin xyz="0.0 0.0 ${shoulder_height}" rpy="0.0 0.0 0.0" />
       <axis xyz="0 0 1" />
-      <xacro:unless value="${joint_limited}">
+      <xacro:unless value="$(arg joint_limited)">
         <limit lower="${-2.0 * pi}" upper="${2.0 * pi}" effort="330.0" velocity="2.16"/>
       </xacro:unless>
-      <xacro:if value="${joint_limited}">
+      <xacro:if value="$(arg joint_limited)">
         <limit lower="${-pi}" upper="${pi}" effort="330.0" velocity="2.16"/>
       </xacro:if>
@@ -109,8 +109,8 @@
       <origin xyz="0.0 ${shoulder_offset} 0.0" rpy="0.0 ${pi / 2.0} 0.0" />
       <axis xyz="0 1 0" />
-      <xacro:unless value="${joint_limited}">
+      <xacro:unless value="$(arg joint_limited)">
         <limit lower="${-2.0 * pi}" upper="${2.0 * pi}" effort="330.0" velocity="2.16"/>
       </xacro:unless>
-      <xacro:if value="${joint_limited}">
+      <xacro:if value="$(arg joint_limited)">
         <limit lower="${-pi}" upper="${pi}" effort="330.0" velocity="2.16"/>
       </xacro:if>
@@ -140,8 +140,8 @@
       <origin xyz="0.0 ${elbow_offset} ${upper_arm_length}" rpy="0.0 0.0 0.0" />
       <axis xyz="0 1 0" />
-      <xacro:unless value="${joint_limited}">
+      <xacro:unless value="$(arg joint_limited)">
         <limit lower="${-2.0 * pi}" upper="${2.0 * pi}" effort="150.0" velocity="3.15"/>
       </xacro:unless>
-      <xacro:if value="${joint_limited}">
+      <xacro:if value="$(arg joint_limited)">
         <limit lower="${-pi}" upper="${pi}" effort="150.0" velocity="3.15"/>
       </xacro:if>
@@ -171,8 +171,8 @@
       <origin xyz="0.0 0.0 ${forearm_length}" rpy="0.0 ${pi / 2.0} 0.0" />
       <axis xyz="0 1 0" />
-      <xacro:unless value="${joint_limited}">
+      <xacro:unless value="$(arg joint_limited)">
         <limit lower="${-2.0 * pi}" upper="${2.0 * pi}" effort="54.0" velocity="3.2"/>
       </xacro:unless>
-      <xacro:if value="${joint_limited}">
+      <xacro:if value="$(arg joint_limited)">
         <limit lower="${-pi}" upper="${pi}" effort="54.0" velocity="3.2"/>
       </xacro:if>
@@ -202,8 +202,8 @@
       <origin xyz="0.0 ${wrist_1_length} 0.0" rpy="0.0 0.0 0.0" />
       <axis xyz="0 0 1" />
-      <xacro:unless value="${joint_limited}">
+      <xacro:unless value="$(arg joint_limited)">
         <limit lower="${-2.0 * pi}" upper="${2.0 * pi}" effort="54.0" velocity="3.2"/>
       </xacro:unless>
-      <xacro:if value="${joint_limited}">
+      <xacro:if value="$(arg joint_limited)">
         <limit lower="${-pi}" upper="${pi}" effort="54.0" velocity="3.2"/>
       </xacro:if>
@@ -233,8 +233,8 @@
       <origin xyz="0.0 0.0 ${wrist_2_length}" rpy="0.0 0.0 0.0" />
       <axis xyz="0 1 0" />
-      <xacro:unless value="${joint_limited}">
+      <xacro:unless value="$(arg joint_limited)">
         <limit lower="${-2.0 * pi}" upper="${2.0 * pi}" effort="54.0" velocity="3.2"/>
       </xacro:unless>
-      <xacro:if value="${joint_limited}">
+      <xacro:if value="$(arg joint_limited)">
         <limit lower="${-pi}" upper="${pi}" effort="54.0" velocity="3.2"/>
       </xacro:if>
@@ -272,10 +272,7 @@
       </collision>
     </link>
-    <xacro:if value="$(arg use_effort_interface)">
-      <xacro:ur_arm_transmission prefix="${prefix}" joint_interface="EffortJointInterface" />
-    </xacro:if>
-    <xacro:unless value="$(arg use_effort_interface)">
-      <xacro:ur_arm_transmission prefix="${prefix}" joint_interface="PositionJointInterface" />
-    </xacro:unless>
+    <!-- setup transmissions -->
+    <xacro:ur_arm_transmission prefix="${prefix}" />
+    <!-- instantiate the arm -->
     <xacro:ur_arm_gazebo prefix="${prefix}" />
     <!-- ROS base_link to UR 'Base' Coordinates transform -->

File: ur_description/urdf/ur10_robot.urdf.xacro (robot description, xacro)
@@ -7,5 +7,5 @@
   <xacro:include filename="$(find ur_description)/urdf/ur10.urdf.xacro" />
   <!-- arm -->
-  <xacro:ur10_robot prefix="" joint_limited="false"/>
+  <xacro:ur10_robot prefix="" />
   <link name="world" />
   <joint name="world_joint" type="fixed">
